Commit message: Add lifting platform and finalize Gazebo model

File: src/tugger_description/urdf/tugger.urdf.xacro (robot description, xacro)
@@ -298,3 +298,46 @@
             rpy="0 0 0"/>
   </joint>
+  <!-- LIFTING PLATFORM -->
+  <link name="lift_platform_link">
+    <visual>
+      <geometry>
+        <box size="0.50 0.32 0.015"/>
+      </geometry>
+      <material name="gap_dark"/>
+    </visual>
+    <collision>
+      <geometry>
+        <box size="0.50 0.32 0.015"/>
+      </geometry>
+    </collision>
+    <inertial>
+      <mass value="3.0"/>
+      <inertia
+        ixx="0.02566"
+        ixy="0"
+        ixz="0"
+        iyy="0.06256"
+        iyz="0"
+        izz="0.08810"/>
+    </inertial>
+  </link>
+  <joint name="lift_joint"
+         type="prismatic">
+    <parent link="base_link"/>
+    <child link="lift_platform_link"/>
+    <!--
+      Lowered position:
+      upper body top = 0.1225 m
+      platform thickness = 0.015 m
+      platform center = 0.1300 m
+    -->
+    <origin xyz="0 0 0.130"
+            rpy="0 0 0"/>
+    <axis xyz="0 0 1"/>
+    <limit
+      lower="0.0"
+      upper="0.040"
+      effort="2000"
+      velocity="0.05"/>
+  </joint>
 </robot>

Commit message: Add ROS 2 control and four-wheel steering actuation

File: src/tugger_description/urdf/tugger.urdf.xacro (robot description, xacro)
@@ -341,3 +341,37 @@
       velocity="0.05"/>
   </joint>
+  <!-- ROS 2 CONTROL -->
+  <ros2_control name="GazeboSimSystem" type="system">
+    <hardware>
+      <plugin>gz_ros2_control/GazeboSimSystem</plugin>
+    </hardware>
+    <joint name="front_left_steering_joint">
+      <command_interface name="position"/>
+      <state_interface name="position"/>
+      <state_interface name="velocity"/>
+    </joint>
+    <joint name="front_right_steering_joint">
+      <command_interface name="position"/>
+      <state_interface name="position"/>
+      <state_interface name="velocity"/>
+    </joint>
+    <joint name="rear_left_steering_joint">
+      <command_interface name="position"/>
+      <state_interface name="position"/>
+      <state_interface name="velocity"/>
+    </joint>
+    <joint name="rear_right_steering_joint">
+      <command_interface name="position"/>
+      <state_interface name="position"/>
+      <state_interface name="velocity"/>
+    </joint>
+  </ros2_control>
+  <!-- GAZEBO ROS 2 CONTROL -->
+  <gazebo>
+    <plugin
+      filename="gz_ros2_control-system"
+      name="gz_ros2_control::GazeboSimROS2ControlPlugin">
+      <parameters>$(find tugger_gazebo)/config/controllers.yaml</parameters>
+    </plugin>
+  </gazebo>
 </robot>

Commit message: Add four-wheel steering and rear traction control

File: src/tugger_description/urdf/tugger.urdf.xacro (robot description, xacro)
@@ -366,4 +366,15 @@
       <state_interface name="velocity"/>
     </joint>
+    <!-- Rear-wheel-drive traction interfaces -->
+    <joint name="rear_left_wheel_joint">
+      <command_interface name="velocity"/>
+      <state_interface name="position"/>
+      <state_interface name="velocity"/>
+    </joint>
+    <joint name="rear_right_wheel_joint">
+      <command_interface name="velocity"/>
+      <state_interface name="position"/>
+      <state_interface name="velocity"/>
+    </joint>
   </ros2_control>
   <!-- GAZEBO ROS 2 CONTROL -->

Commit message: Fix wheel contact physics for smooth 4WS turning

File: src/tugger_description/urdf/tugger.urdf.xacro (robot description, xacro)
@@ -159,4 +159,16 @@
     </joint>
   </xacro:macro>
+  <!-- GAZEBO WHEEL CONTACT / FRICTION -->
+  <xacro:macro name="wheel_gazebo_friction" params="prefix">
+    <gazebo reference="${prefix}_wheel_link">
+      <mu1>1.0</mu1>
+      <mu2>0.20</mu2>
+      <fdir1>1 0 0</fdir1>
+    </gazebo>
+  </xacro:macro>
+  <xacro:wheel_gazebo_friction prefix="front_left"/>
+  <xacro:wheel_gazebo_friction prefix="front_right"/>
+  <xacro:wheel_gazebo_friction prefix="rear_left"/>
+  <xacro:wheel_gazebo_friction prefix="rear_right"/>
   <!-- FOUR-WHEEL STEERING -->
   <xacro:steered_wheel
@@ -228,4 +240,51 @@
             rpy="0 0 0"/>
   </joint>
+  <!-- GAZEBO LIDAR SENSORS -->
+  <gazebo reference="front_left_lidar_link">
+    <sensor name="front_left_lidar_sensor" type="gpu_lidar">
+      <always_on>true</always_on>
+      <update_rate>15</update_rate>
+      <topic>front_left/scan</topic>
+      <gz_frame_id>front_left_lidar_link</gz_frame_id>
+      <lidar>
+        <scan>
+          <horizontal>
+            <samples>720</samples>
+            <resolution>1</resolution>
+            <min_angle>-3.14159265</min_angle>
+            <max_angle>3.14159265</max_angle>
+          </horizontal>
+        </scan>
+        <range>
+          <min>0.08</min>
+          <max>20.0</max>
+          <resolution>0.01</resolution>
+        </range>
+      </lidar>
+    </sensor>
+  </gazebo>
+  <gazebo reference="rear_right_lidar_link">
+    <sensor name="rear_right_lidar_sensor" type="gpu_lidar">
+      <always_on>true</always_on>
+      <update_rate>15</update_rate>
+      <topic>rear_right/scan</topic>
+      <gz_frame_id>rear_right_lidar_link</gz_frame_id>
+      <lidar>
+        <scan>
+          <horizontal>
+            <samples>720</samples>
+            <resolution>1</resolution>
+            <min_angle>-3.14159265</min_angle>
+            <max_angle>3.14159265</max_angle>
+          </horizontal>
+        </scan>
+        <range>
+          <min>0.08</min>
+          <max>20.0</max>
+          <resolution>0.01</resolution>
+        </range>
+      </lidar>
+    </sensor>
+  </gazebo>
   <!-- FRONT CAMERA -->
   <link name="front_camera_link">

Commit message: Add camera simulation and SLAM integration

File: src/tugger_description/urdf/tugger.urdf.xacro (robot description, xacro)
@@ -516,4 +516,18 @@
       <state_interface name="velocity"/>
     </joint>
+    <!-- Passive front-wheel state interfaces -->
+    <joint name="front_left_wheel_joint">
+      <state_interface name="position"/>
+      <state_interface name="velocity"/>
+    </joint>
+    <joint name="front_right_wheel_joint">
+      <state_interface name="position"/>
+      <state_interface name="velocity"/>
+    </joint>
+    <!-- Lift state interface -->
+    <joint name="lift_joint">
+      <state_interface name="position"/>
+      <state_interface name="velocity"/>
+    </joint>
     <!-- Rear-wheel-drive traction interfaces -->
     <joint name="rear_left_wheel_joint">
